File: pcb/eightbyeight.sch (EAGLE design)
At the start: 164 parts, among them CON1 USB_MICROSMT+THRUHULE, Q1 16MHz, SW1 SWITCH_SPDT, SW2 BRIGHTNESS, U1 MK20DN64VFM5, U10 FDG6316P, U11 FDG6316P, U12 FDG6316P, U2 ICN2026, U3 74138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

Commit message: Small updates from further testing
Parts:
- R1: value 1.8k 1% -> 1.6k 1%
- R12, R23, R25, R26, R27: value 47k -> 10k
Other:
- note added: "ESP826 Boot Select UART Download: GPIO15 Low, GPIO0 Low, GPIO2 High Flash Boot: GPIO15 Low, GPIO0 Hight, GPIO2 High Note: The ESP8266 needs strong pullup/down resistors on the boot select lines. 10k is stable, 47k is marginal, and 100k is unreliable."
- note removed: "ESP826 Boot Select UART Download: GPIO15 Low, GPIO0 Low, GPIO2 High Flash Boot: GPIO15 Low, GPIO0 Hight, GPIO2 High"
- moved on the sheet: R12, R23, R25
Changed lines of the file:
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@@
 <part name="GND2" library="SparkFun-Aesthetics" deviceset="GND" device=""/>
 <part name="C7" library="adafruit" deviceset="C-US" device="C0402" value="100nF"/>
-<part name="R1" library="adafruit" deviceset="R-US_" device="R0402" value="1.8k 1%"/>
+<part name="R1" library="adafruit" deviceset="R-US_" device="R0402" value="1.6k 1%"/>
 <part name="GND3" library="SparkFun-Aesthetics" deviceset="GND" device=""/>
 <part name="GND4" library="SparkFun-Aesthetics" deviceset="GND" device=""/>
@@
 <part name="GND32" library="SparkFun-Aesthetics" deviceset="GND" device=""/>
 <part name="GND33" library="SparkFun-Aesthetics" deviceset="GND" device=""/>
-<part name="R23" library="adafruit" deviceset="R-US_" device="R0402" value="47k"/>
-<part name="R25" library="adafruit" deviceset="R-US_" device="R0402" value="47k"/>
+<part name="R23" library="adafruit" deviceset="R-US_" device="R0402" value="10k"/>
+<part name="R25" library="adafruit" deviceset="R-US_" device="R0402" value="10k"/>
 <part name="3V16" library="supply1" deviceset="+3V3" device=""/>
 <part name="GND34" library="supply1" deviceset="GND" device=""/>
 <part name="FRAME5" library="frames" deviceset="A3L-LOC" device=""/>
-<part name="R26" library="adafruit" deviceset="R-US_" device="R0402" value="47k"/>
-<part name="R27" library="adafruit" deviceset="R-US_" device="R0402" value="47k"/>
+<part name="R26" library="adafruit" deviceset="R-US_" device="R0402" value="10k"/>
+<part name="R27" library="adafruit" deviceset="R-US_" device="R0402" value="10k"/>
 <part name="3V17" library="supply1" deviceset="+3V3" device=""/>
 <part name="3V18" library="supply1" deviceset="+3V3" device=""/>
@@
 <part name="ANALOG_IN" library="testpad" deviceset="PTR1" device="B2,54"/>
 <part name="3V3" library="supply1" deviceset="+3V3" device=""/>
-<part name="R12" library="adafruit" deviceset="R-US_" device="R0402" value="47k"/>
+<part name="R12" library="adafruit" deviceset="R-US_" device="R0402" value="10k"/>
 <part name="TP16" library="testpad" deviceset="PTR1" device="B1,27"/>
 <part name="R21" library="adafruit" deviceset="R-US_" device="R0402" value="47k"/>
@@
 Revision D:
 -Replace ARM JTAG connector with test points for automated programming
--Change value of pullup resistors from 10k to 47k
 -Update filter caps for 3.3V regulator
 -Add test pads for production
@@
 <wire x1="246.38" y1="175.26" x2="246.38" y2="251.46" width="0.4064" layer="94"/>
 <wire x1="10.16" y1="175.26" x2="246.38" y2="175.26" width="0.4064" layer="94"/>
-<text x="160.02" y="228.6" size="1.778" layer="91">ESP826 Boot Select
+<text x="157.48" y="223.52" size="1.778" layer="91">ESP826 Boot Select
 UART Download:
 GPIO15 Low, GPIO0 Low, GPIO2 High
 Flash Boot:
-GPIO15 Low, GPIO0 Hight, GPIO2 High</text>
+GPIO15 Low, GPIO0 Hight, GPIO2 High
+Note: The ESP8266 needs strong pullup/down resistors
+on the boot select lines. 10k is stable, 47k is marginal,
+and 100k is unreliable.</text>
 <text x="15.24" y="157.48" size="1.778" layer="91">Note: The I2C bus runs at 100KHz</text>
 <text x="15.24" y="162.56" size="2.54" layer="94">I2C pullups</text>
@@
 </instance>
 <instance part="GND23" gate="1" x="50.8" y="185.42"/>
-<instance part="R23" gate="G$1" x="226.06" y="208.28" smashed="yes" rot="R90">
-<attribute name="NAME" x="225.0694" y="202.692" size="1.778" layer="95" rot="R90"/>
-<attribute name="VALUE" x="225.044" y="211.328" size="1.778" layer="96" rot="R90"/>
-</instance>
-<instance part="R25" gate="G$1" x="203.2" y="193.04" smashed="yes" rot="R90">
-<attribute name="NAME" x="202.2094" y="187.452" size="1.778" layer="95" rot="R90"/>
-<attribute name="VALUE" x="202.184" y="196.088" size="1.778" layer="96" rot="R90"/>
-</instance>
-<instance part="3V16" gate="G$1" x="226.06" y="218.44" smashed="yes">
-<attribute name="VALUE" x="223.52" y="219.71" size="1.778" layer="96"/>
-</instance>
-<instance part="GND34" gate="1" x="203.2" y="182.88"/>
+<instance part="R23" gate="G$1" x="226.06" y="205.74" smashed="yes" rot="R90">
+<attribute name="NAME" x="225.0694" y="200.152" size="1.778" layer="95" rot="R90"/>
+<attribute name="VALUE" x="225.044" y="208.788" size="1.778" layer="96" rot="R90"/>
+</instance>
+<instance part="R25" gate="G$1" x="203.2" y="190.5" smashed="yes" rot="R90">
+<attribute name="NAME" x="202.2094" y="184.912" size="1.778" layer="95" rot="R90"/>
+<attribute name="VALUE" x="202.184" y="193.548" size="1.778" layer="96" rot="R90"/>
+</instance>
+<instance part="3V16" gate="G$1" x="226.06" y="215.9" smashed="yes">
+<attribute name="VALUE" x="223.52" y="217.17" size="1.778" layer="96"/>
+</instance>
+<instance part="GND34" gate="1" x="203.2" y="180.34"/>
 <instance part="R17" gate="G$1" x="20.32" y="134.62" rot="R90"/>
 <instance part="R18" gate="G$1" x="25.4" y="134.62" rot="R90"/>
@@
 <instance part="5" gate="G$1" x="287.02" y="226.06" rot="R90"/>
 <instance part="ANALOG_IN" gate="G$1" x="287.02" y="210.82" rot="R90"/>
-<instance part="3V3" gate="G$1" x="180.34" y="218.44" smashed="yes">
-<attribute name="VALUE" x="177.8" y="219.71" size="1.778" layer="96"/>
-</instance>
-<instance part="R12" gate="G$1" x="180.34" y="208.28" smashed="yes" rot="R90">
-<attribute name="NAME" x="179.3494" y="202.692" size="1.778" layer="95" rot="R90"/>
-<attribute name="VALUE" x="179.324" y="211.328" size="1.778" layer="96" rot="R90"/>
+<instance part="3V3" gate="G$1" x="180.34" y="215.9" smashed="yes">
+<attribute name="VALUE" x="177.8" y="217.17" size="1.778" layer="96"/>
+</instance>
+<instance part="R12" gate="G$1" x="180.34" y="205.74" smashed="yes" rot="R90">
+<attribute name="NAME" x="179.3494" y="200.152" size="1.778" layer="95" rot="R90"/>
+<attribute name="VALUE" x="179.324" y="208.788" size="1.778" layer="96" rot="R90"/>
 </instance>
 <instance part="3.3V" gate="G$1" x="287.02" y="198.12" rot="R90"/>
@@
 <pinref part="R25" gate="G$1" pin="1"/>
 <pinref part="GND34" gate="1" pin="GND"/>
-<wire x1="203.2" y1="187.96" x2="203.2" y2="185.42" width="0.1524" layer="91"/>
+<wire x1="203.2" y1="185.42" x2="203.2" y2="182.88" width="0.1524" layer="91"/>
 </segment>
 <segment>
@@
 <pinref part="3V16" gate="G$1" pin="+3V3"/>
 <pinref part="R23" gate="G$1" pin="2"/>
-<wire x1="226.06" y1="215.9" x2="226.06" y2="213.36" width="0.1524" layer="91"/>
+<wire x1="226.06" y1="213.36" x2="226.06" y2="210.82" width="0.1524" layer="91"/>
 </segment>
 <segment>
@@
 <pinref part="3V3" gate="G$1" pin="+3V3"/>
 <pinref part="R12" gate="G$1" pin="2"/>
-<wire x1="180.34" y1="215.9" x2="180.34" y2="213.36" width="0.1524" layer="91"/>
+<wire x1="180.34" y1="213.36" x2="180.34" y2="210.82" width="0.1524" layer="91"/>
 </segment>
 <segment>
@@
 </segment>
 <segment>
-<wire x1="180.34" y1="200.66" x2="162.56" y2="200.66" width="0.1524" layer="91"/>
+<wire x1="180.34" y1="198.12" x2="162.56" y2="198.12" width="0.1524" layer="91"/>
 <pinref part="R12" gate="G$1" pin="1"/>
-<wire x1="180.34" y1="203.2" x2="180.34" y2="200.66" width="0.1524" layer="91"/>
-<label x="162.56" y="200.66" size="1.778" layer="95"/>
+<wire x1="180.34" y1="200.66" x2="180.34" y2="198.12" width="0.1524" layer="91"/>
+<label x="162.56" y="198.12" size="1.778" layer="95"/>
 </segment>
 <segment>
@@
 <segment>
 <pinref part="R23" gate="G$1" pin="1"/>
-<wire x1="226.06" y1="203.2" x2="226.06" y2="200.66" width="0.1524" layer="91"/>
-<wire x1="226.06" y1="200.66" x2="210.82" y2="200.66" width="0.1524" layer="91"/>
-<label x="210.82" y="200.66" size="1.778" layer="95"/>
+<wire x1="226.06" y1="200.66" x2="226.06" y2="198.12" width="0.1524" layer="91"/>
+<wire x1="226.06" y1="198.12" x2="210.82" y2="198.12" width="0.1524" layer="91"/>
+<label x="210.82" y="198.12" size="1.778" layer="95"/>
 </segment>
 <segment>
@@
 <segment>
 <pinref part="R25" gate="G$1" pin="2"/>
-<wire x1="187.96" y1="200.66" x2="203.2" y2="200.66" width="0.1524" layer="91"/>
-<wire x1="203.2" y1="200.66" x2="203.2" y2="198.12" width="0.1524" layer="91"/>
-<label x="187.96" y="200.66" size="1.778" layer="95"/>
-</segment>
-</net>
+<wire x1="187.96" y1="198.12" x2="203.2" y2="198.12" width="0.1524" layer="91"/>
+<wire x1="203.2" y1="198.12" x2="203.2" y2="195.58" width="0.1524" layer="91"/>
+<label x="187.96" y="198.12" size="1.778" layer="95"/>
+</segment>
+</net>

Commit message: RevE.A
Parts:
- removed 16, 3.3V, 5, ANALOG_IN, GROUND: PTR1B2,54, testpad:PTR1B2,54
- added U$10, U$2, U$6, U$9: TEST_POINT, DevicesToMerge:TEST_POINT
- R13, R14, R15, R16, R2, R3, R4, R5: value 2k -> 4.7k
- R21, R6: value 47k -> 10k
- renumbered BAT to J2, CON1 to J1, U$8 to U7
Connections:
- net +3V3: now also U$10.P$1; no longer 3.3V.TP
- net ESP_GPIO16: now also U$9.P$1; no longer 16.TP
- net ESP_TOUT: no longer ANALOG_IN.TP
- net EXP_GPIO5: now also U$6.P$1; no longer 5.TP
- net GND: now also U$2.P$1; no longer GROUND.TP
