File: pcb/testcard/raspberrypi-testcard.brd (EAGLE design)
At the start: 115 x 66 mm, 53 parts, among them IC9 DS1307SO08, J1 USB_MICROSMT+THRUHULE, J2 USB-A, Q3 32.768kHz, 12.5pF, SW2 BRIGHTNESS, U1 ADS1015, U10 N-CHANNEL-MOSFET-BSS138, U12 N-CHANNEL-MOSFET-BSS138, U2 ADS1015, U3 INA219BIDCNT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

Commit message: Update test card pcb notes
Parts:
- R10: value 0.1/1% (PT2512FK-070R1L) -> 50/1% (PT2512FK-070R1L)
Connections:
- net 3.3V: no longer C1.1, C3.1, U1.8, U2.1, U2.8
- net 5V: now also C1.1, C3.1, U1.8, U2.1, U2.8
Routing:
- net 3.3V: track 223.6 -> 183.9 mm
- net 5V: track 161.5 -> 179.7 mm
- net AIN7: track 66.0 -> 56.8 mm
Other:
- board text added: "0x40"
- board text added: "0x48"
- board text added: "0x49"
- board text added: "0x68"
