File: pcb/testcard/raspberrypi-testcard.sch (EAGLE design)
At the start: 53 parts, among them IC9 DS1307SO08, J1 USB_MICROSMT+THRUHULE, J2 USB-A, Q3 32.768kHz, 12.5pF, SW2 BRIGHTNESS, U1 ADS1015, U10 N-CHANNEL-MOSFET-BSS138, U12 N-CHANNEL-MOSFET-BSS138, U2 ADS1015, U3 INA219BIDCNT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

Commit message: Update test card pcb notes
Parts:
- R10: value 0.1/1% (PT2512FK-070R1L) -> 50/1% (PT2512FK-070R1L)
Connections:
- net 3.3V: no longer C1.1, C3.1, U1.VDD, U2.ADDR, U2.VDD
- net 5V: now also C1.1, C3.1, U1.VDD, U2.ADDR, U2.VDD
Other:
- note added: "FAIL LED"
- note added: "GP10"
- note added: "GP11"
- note added: "GP7"
- note added: "GP9"
- note added: "PASS LED"
- note added: "POWER_FULL"
- note added: "POWER_LIMITED"
- note added: "Revision Notes/Changelog Revision A: -Initial version TODO: -Add fuse on DUT power -Switch digital test pins to I/O expander for protection, drive strength, and 3.3/5v configuration -Move LEDs off of serial line, break out as FTDI header -Use 5V for ADC power -Add buffer for JTAG/ICSP -Determine if JTAG requires hardware SPI, and if not move off of SPI and break out SPI -Fix battery connector"
- note added: "START BUTTON"
- note added: "USB RELAY"
- note removed: "Revision Notes/Changelog Revision A: -Initial version"
Changed lines of the file:
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@@
 <part name="SUPPLY1" library="SparkFun-Aesthetics" deviceset="5V" device=""/>
 <part name="SUPPLY2" library="SparkFun-Aesthetics" deviceset="3.3V" device=""/>
-<part name="SUPPLY3" library="SparkFun-Aesthetics" deviceset="3.3V" device=""/>
-<part name="SUPPLY4" library="SparkFun-Aesthetics" deviceset="3.3V" device=""/>
-<part name="SUPPLY5" library="SparkFun-Aesthetics" deviceset="3.3V" device=""/>
 <part name="J1" library="blinkinlabs" deviceset="USB_MICRO" device="SMT+THRUHULE"/>
 <part name="U$2" library="blinkinlabs" deviceset="RELAY" device=""/>
@@
 <part name="GND14" library="supply1" deviceset="GND" device=""/>
 <part name="GND15" library="supply1" deviceset="GND" device=""/>
-<part name="SUPPLY9" library="SparkFun-Aesthetics" deviceset="3.3V" device=""/>
-<part name="SUPPLY10" library="SparkFun-Aesthetics" deviceset="3.3V" device=""/>
 <part name="R17" library="adafruit" deviceset="R-US_" device="R0402" value="4.7k"/>
 <part name="R18" library="adafruit" deviceset="R-US_" device="R0402" value="4.7k"/>
@@
 <part name="GND25" library="supply1" deviceset="GND" device=""/>
 <part name="C2" library="adafruit" deviceset="C-US" device="C0402" value="100nF"/>
-<part name="R10" library="microbuilder" deviceset="RESISTOR" device="2512" value="0.1/1% (PT2512FK-070R1L)"/>
+<part name="R10" library="microbuilder" deviceset="RESISTOR" device="2512" value="50/1% (PT2512FK-070R1L)"/>
 <part name="U9" library="GeekAmmo" deviceset="P-CHANNEL-MOSFET" device=""/>
 <part name="U10" library="GeekAmmo" deviceset="N-CHANNEL-MOSFET" device="-BSS138"/>
@@
 <part name="SW2" library="blinkinlabs" deviceset="BUTTON_MOMENTARY_GROUND" device="" value="BRIGHTNESS"/>
 <part name="GND32" library="supply1" deviceset="GND" device=""/>
+<part name="SUPPLY3" library="SparkFun-Aesthetics" deviceset="5V" device=""/>
+<part name="SUPPLY5" library="SparkFun-Aesthetics" deviceset="5V" device=""/>
+<part name="SUPPLY9" library="SparkFun-Aesthetics" deviceset="5V" device=""/>
+<part name="SUPPLY10" library="SparkFun-Aesthetics" deviceset="5V" device=""/>
+<part name="SUPPLY4" library="SparkFun-Aesthetics" deviceset="5V" device=""/>
 </parts>
 <sheets>
@@
 <text x="17.78" y="325.12" size="3.81" layer="91" align="top-left">Revision Notes/Changelog
 Revision A:
--Initial version</text>
+-Initial version
+TODO:
+-Add fuse on DUT power
+-Switch digital test pins to I/O expander for protection, drive strength,
+  and 3.3/5v configuration
+-Move LEDs off of serial line, break out as FTDI header
+-Use 5V for ADC power
+-Add buffer for JTAG/ICSP
+-Determine if JTAG requires hardware SPI, and if not move off of SPI
+  and break out SPI
+-Fix battery connector</text>
 <text x="129.54" y="358.14" size="10.16" layer="91" align="bottom-center">Raspberry Pi Test driver</text>
 <text x="129.54" y="345.44" size="6.4516" layer="91" align="bottom-center">Copyright 2016 Blinkinlabs, LLC</text>
@@
 <wire x1="678.18" y1="142.24" x2="678.18" y2="251.46" width="0.4064" layer="94"/>
 <wire x1="561.34" y1="142.24" x2="678.18" y2="142.24" width="0.4064" layer="94"/>
+<text x="119.38" y="187.96" size="1.778" layer="91">GP11</text>
+<text x="119.38" y="185.42" size="1.778" layer="91">GP9</text>
+<text x="119.38" y="182.88" size="1.778" layer="91">GP10</text>
+<text x="119.38" y="177.8" size="1.778" layer="91">GP7</text>
+<text x="119.38" y="180.34" size="1.778" layer="91">START BUTTON</text>
+<text x="119.38" y="167.64" size="1.778" layer="91">USB RELAY</text>
+<text x="119.38" y="195.58" size="1.778" layer="91">PASS LED</text>
+<text x="119.38" y="193.04" size="1.778" layer="91">FAIL LED</text>
+<text x="119.38" y="154.94" size="1.778" layer="91">POWER_LIMITED</text>
+<text x="119.38" y="160.02" size="1.778" layer="91">POWER_FULL</text>
 </plain>
 <instances>
@@
 <instance part="SUPPLY1" gate="G$1" x="58.42" y="208.28"/>
 <instance part="SUPPLY2" gate="G$1" x="50.8" y="208.28"/>
-<instance part="SUPPLY3" gate="G$1" x="101.6" y="-35.56"/>
-<instance part="SUPPLY4" gate="G$1" x="139.7" y="-99.06"/>
-<instance part="SUPPLY5" gate="G$1" x="101.6" y="-93.98"/>
 <instance part="J1" gate="G$1" x="198.12" y="-55.88"/>
 <instance part="U$2" gate="G$1" x="223.52" y="-76.2" rot="R90"/>
@@
 <instance part="GND14" gate="1" x="20.32" y="-60.96"/>
 <instance part="GND15" gate="1" x="20.32" y="-114.3"/>
-<instance part="SUPPLY9" gate="G$1" x="20.32" y="-99.06"/>
-<instance part="SUPPLY10" gate="G$1" x="20.32" y="-45.72"/>
 <instance part="R17" gate="G$1" x="33.02" y="50.8" rot="R90"/>
 <instance part="R18" gate="G$1" x="38.1" y="50.8" rot="R90"/>
@@
 </instance>
 <instance part="GND32" gate="1" x="464.82" y="-83.82"/>
+<instance part="SUPPLY3" gate="G$1" x="101.6" y="-35.56"/>
+<instance part="SUPPLY5" gate="G$1" x="20.32" y="-45.72"/>
+<instance part="SUPPLY9" gate="G$1" x="20.32" y="-99.06"/>
+<instance part="SUPPLY10" gate="G$1" x="101.6" y="-93.98"/>
+<instance part="SUPPLY4" gate="G$1" x="139.7" y="-99.06"/>
 </instances>
 <busses>
@@
 <junction x="622.3" y="215.9"/>
 </segment>
+<segment>
+<pinref part="U1" gate="G$1" pin="VDD"/>
+<wire x1="101.6" y1="-35.56" x2="101.6" y2="-38.1" width="0.1524" layer="91"/>
+<pinref part="SUPPLY3" gate="G$1" pin="5V"/>
+</segment>
+<segment>
+<pinref part="C3" gate="G$1" pin="1"/>
+<wire x1="20.32" y1="-45.72" x2="20.32" y2="-48.26" width="0.1524" layer="91"/>
+<pinref part="SUPPLY5" gate="G$1" pin="5V"/>
+</segment>
+<segment>
+<pinref part="C1" gate="G$1" pin="1"/>
+<wire x1="20.32" y1="-99.06" x2="20.32" y2="-101.6" width="0.1524" layer="91"/>
+<pinref part="SUPPLY9" gate="G$1" pin="5V"/>
+</segment>
+<segment>
+<pinref part="U2" gate="G$1" pin="VDD"/>
+<wire x1="101.6" y1="-93.98" x2="101.6" y2="-96.52" width="0.1524" layer="91"/>
+<pinref part="SUPPLY10" gate="G$1" pin="5V"/>
+</segment>
+<segment>
+<pinref part="U2" gate="G$1" pin="ADDR"/>
+<wire x1="137.16" y1="-111.76" x2="139.7" y2="-111.76" width="0.1524" layer="91"/>
+<wire x1="139.7" y1="-111.76" x2="139.7" y2="-99.06" width="0.1524" layer="91"/>
+<pinref part="SUPPLY4" gate="G$1" pin="5V"/>
+</segment>
 </net>
 <net name="3.3V" class="1">
@@
 </segment>
 <segment>
-<pinref part="U1" gate="G$1" pin="VDD"/>
-<pinref part="SUPPLY3" gate="G$1" pin="3.3V"/>
-<wire x1="101.6" y1="-35.56" x2="101.6" y2="-38.1" width="0.1524" layer="91"/>
-</segment>
-<segment>
-<pinref part="U2" gate="G$1" pin="ADDR"/>
-<wire x1="137.16" y1="-111.76" x2="139.7" y2="-111.76" width="0.1524" layer="91"/>
-<wire x1="139.7" y1="-111.76" x2="139.7" y2="-99.06" width="0.1524" layer="91"/>
-<pinref part="SUPPLY4" gate="G$1" pin="3.3V"/>
-</segment>
-<segment>
-<pinref part="U2" gate="G$1" pin="VDD"/>
-<pinref part="SUPPLY5" gate="G$1" pin="3.3V"/>
-<wire x1="101.6" y1="-93.98" x2="101.6" y2="-96.52" width="0.1524" layer="91"/>
-</segment>
-<segment>
-<pinref part="SUPPLY10" gate="G$1" pin="3.3V"/>
-<pinref part="C3" gate="G$1" pin="1"/>
-<wire x1="20.32" y1="-45.72" x2="20.32" y2="-48.26" width="0.1524" layer="91"/>
-</segment>
-<segment>
-<pinref part="SUPPLY9" gate="G$1" pin="3.3V"/>
-<pinref part="C1" gate="G$1" pin="1"/>
-<wire x1="20.32" y1="-99.06" x2="20.32" y2="-101.6" width="0.1524" layer="91"/>
-</segment>
-<segment>
